File: PCB/Klotz.kicad_pcb (KiCad board)
At the start: 2 copper layers, 120.5 x 85.5 mm, 56 parts, among them SW1 MX_SW_HS, SW10 MX_SW_HS, SW11 MX_SW_HS, SW12 MX_SW_HS, SW13 MX_SW_HS, SW14 MX_SW_HS, SW15 MX_SW_HS, SW16 MX_SW_HS, SW17 MX_SW_HS, SW18 RotaryEncoder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

Commit message: init
Parts:
- removed SW18: RotaryEncoder, Rotary_Encoder:RotaryEncoder_Alps_EC12E_Vertical_H20mm
- added SW19: EVQWGD001, evq:EVQWGD001, F.Cu at (97.3, 101.7)
Routing:
- net ENCB: track 35.1 -> 46.2 mm
- net Net-(BT2-+): track 122.1 -> 118.5 mm
- net col4: track 206.5 -> 202.9 mm
- net row2: track 171.9 -> 168.6 mm
- net +BATT: track 61.6 -> 58.5 mm
- net ENCA: track 42.4 -> 45.0 mm, vias 2 -> 3
- net col3: track 209.9 -> 210.4 mm
- net col1: track 256.8 -> 257.4 mm
- net col0: track 271.0 -> 271.6 mm
- net col2: track 204.6 -> 205.1 mm
- net GND: vias 63 -> 62
