File: PCB/Klotz.kicad_sch (KiCad schematic)
At the start: 55 parts, among them SW1 MX_SW_HS, SW10 MX_SW_HS, SW11 MX_SW_HS, SW12 MX_SW_HS, SW13 MX_SW_HS, SW14 MX_SW_HS, SW15 MX_SW_HS, SW16 MX_SW_HS, SW17 MX_SW_HS, SW18 RotaryEncoder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

Commit message: init
Parts:
- removed SW18: RotaryEncoder, Rotary_Encoder:RotaryEncoder_Alps_EC12E_Vertical_H20mm, symbol Device:RotaryEncoder
- added SW19: EVQWGD001, evq:EVQWGD001, symbol barobord:EVQWGD001
- RSW1: footprint (none) -> KLOTZ:ResetSW
Connections:
- net ENCA: now also SW19.A
- net ENCB: now also SW19.C
- net GND: now also SW19.B
- no-connect marks 5 -> 8
